Commit message: fix: camera urdf for gazebo & rviz

File: src/turtlebot3_descriptions/urdf/turtlebot3_burger_oak_d_pro.urdf (robot description, URDF)
Before this commit: robot turtlebot3_burger, 10 links, 9 joints
Links:
- link oak_d_pro_camera: geometry collision box size=0.1 0.03 0.025; visual mesh filename=package://turtlebot3_descriptions/meshes/sensors/OAK-D-PRO.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 scale=1.0 1.0 1.0
Joints:
- joint joint_oak_d_pro_camera: origin xyz=0.065 0.0 0.11 rpy=1.57 0.0 1.57 -> xyz=-0.13 0.0 0.14 rpy=0.785 0 -1.57
- joint joint_oak_d_pro_color_optical_frame: origin xyz=0.0 0.0 0.0 rpy=-1.5708 0.0 -1.5708 -> xyz=0.0 0.0 0.0 rpy=0.0 0.0 -1.57
- joint joint_oak_d_pro_depth_optical_frame: origin xyz=0.0 0.0 0.0 rpy=-1.5708 0.0 -1.5708 -> xyz=0.0 0.0 0.0 rpy=0 0.0 0.0

Commit message: feat: Add camera to rviz

File: src/turtlebot3_descriptions/urdf/turtlebot3_burger_oak_d_pro.urdf (robot description, URDF)
Before this commit: robot turtlebot3_burger, 10 links, 9 joints
Joints:
- joint joint_oak_d_pro_camera: origin xyz=-0.13 0.0 0.14 rpy=0.785 0 -1.57 -> xyz=-0.13 0.0 0.14 rpy=0.785 0.0 -1.57
- joint joint_oak_d_pro_depth_optical_frame: origin xyz=0.0 0.0 0.0 rpy=0 0.0 0.0 -> xyz=0.0 0.0 0.0 rpy=0.0 0.0 0.0

Commit message: fix: change camera orientation

File: src/turtlebot3_descriptions/urdf/turtlebot3_burger_oak_d_pro.urdf (robot description, URDF)
Before this commit: robot turtlebot3_burger, 10 links, 9 joints
Joints:
- joint joint_oak_d_pro_camera: origin xyz=-0.13 0.0 0.14 rpy=0.785 0.0 -1.57 -> xyz=0.07 0.0 0.14 rpy=0.9 0.0 1.57

Commit message: fix: fix depth part in rviz

File: src/turtlebot3_descriptions/urdf/turtlebot3_burger_oak_d_pro.urdf (robot description, URDF)
Before this commit: robot turtlebot3_burger, 10 links, 9 joints
Joints:
- joint joint_oak_d_pro_depth_optical_frame: origin xyz=0.0 0.0 0.0 rpy=0.0 0.0 0.0 -> xyz=0.0 0.0 0.0 rpy=0 0 -1.57
